File: hardware/RGB_LED_Controller.sch (EAGLE design)
At the start: 16 parts, among them IC2 MEGA8-AI, J2 CON_HEADER_1X04, Q1 MOSFET-NCHANNELFDD8580, Q2 MOSFET-NCHANNELFDD8580, Q4 MOSFET-NCHANNELFDD8580

Commit message: some routing done. PCB modified to 7043
Connections:
- net GND: now also U$4.PIO5
Changed lines of the file:
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@@
 <?xml version="1.0" encoding="utf-8"?>
 <!DOCTYPE eagle SYSTEM "eagle.dtd">
-<eagle version="6.2">
+<eagle version="6.1">
 <drawing>
 <settings>
@@
 <grid distance="0.1" unitdist="inch" unit="inch" style="lines" multiple="1" display="no" altdistance="0.01" altunitdist="inch" altunit="inch"/>
 <layers>
-<layer number="1" name="Top" color="4" fill="1" visible="yes" active="no"/>
-<layer number="2" name="Route2" color="1" fill="3" visible="yes" active="no"/>
-<layer number="3" name="Route3" color="4" fill="3" visible="yes" active="no"/>
-<layer number="4" name="Route4" color="1" fill="4" visible="yes" active="no"/>
-<layer number="5" name="Route5" color="4" fill="4" visible="yes" active="no"/>
-<layer number="6" name="Route6" color="1" fill="8" visible="yes" active="no"/>
-<layer number="7" name="Route7" color="4" fill="8" visible="yes" active="no"/>
-<layer number="8" name="Route8" color="1" fill="2" visible="yes" active="no"/>
-<layer number="9" name="Route9" color="4" fill="2" visible="yes" active="no"/>
-<layer number="10" name="Route10" color="1" fill="7" visible="yes" active="no"/>
-<layer number="11" name="Route11" color="4" fill="7" visible="yes" active="no"/>
-<layer number="12" name="Route12" color="1" fill="5" visible="yes" active="no"/>
-<layer number="13" name="Route13" color="4" fill="5" visible="yes" active="no"/>
-<layer number="14" name="Route14" color="1" fill="6" visible="yes" active="no"/>
-<layer number="15" name="Route15" color="4" fill="6" visible="yes" active="no"/>
-<layer number="16" name="Bottom" color="1" fill="1" visible="yes" active="no"/>
-<layer number="17" name="Pads" color="2" fill="1" visible="yes" active="no"/>
-<layer number="18" name="Vias" color="2" fill="1" visible="yes" active="no"/>
-<layer number="19" name="Unrouted" color="6" fill="1" visible="yes" active="no"/>
-<layer number="20" name="Dimension" color="15" fill="1" visible="yes" active="no"/>
-<layer number="21" name="tPlace" color="7" fill="1" visible="yes" active="no"/>
-<layer number="22" name="bPlace" color="7" fill="1" visible="yes" active="no"/>
-<layer number="23" name="tOrigins" color="15" fill="1" visible="yes" active="no"/>
-<layer number="24" name="bOrigins" color="15" fill="1" visible="yes" active="no"/>
-<layer number="25" name="tNames" color="7" fill="1" visible="yes" active="no"/>
-<layer number="26" name="bNames" color="7" fill="1" visible="yes" active="no"/>
-<layer number="27" name="tValues" color="7" fill="1" visible="yes" active="no"/>
-<layer number="28" name="bValues" color="7" fill="1" visible="yes" active="no"/>
+<layer number="1" name="Top" color="4" fill="1" visible="no" active="no"/>
+<layer number="2" name="Route2" color="1" fill="3" visible="no" active="no"/>
+<layer number="3" name="Route3" color="4" fill="3" visible="no" active="no"/>
+<layer number="4" name="Route4" color="1" fill="4" visible="no" active="no"/>
+<layer number="5" name="Route5" color="4" fill="4" visible="no" active="no"/>
+<layer number="6" name="Route6" color="1" fill="8" visible="no" active="no"/>
+<layer number="7" name="Route7" color="4" fill="8" visible="no" active="no"/>
+<layer number="8" name="Route8" color="1" fill="2" visible="no" active="no"/>
+<layer number="9" name="Route9" color="4" fill="2" visible="no" active="no"/>
+<layer number="10" name="Route10" color="1" fill="7" visible="no" active="no"/>
+<layer number="11" name="Route11" color="4" fill="7" visible="no" active="no"/>
+<layer number="12" name="Route12" color="1" fill="5" visible="no" active="no"/>
+<layer number="13" name="Route13" color="4" fill="5" visible="no" active="no"/>
+<layer number="14" name="Route14" color="1" fill="6" visible="no" active="no"/>
+<layer number="15" name="Route15" color="4" fill="6" visible="no" active="no"/>
+<layer number="16" name="Bottom" color="1" fill="1" visible="no" active="no"/>
+<layer number="17" name="Pads" color="2" fill="1" visible="no" active="no"/>
+<layer number="18" name="Vias" color="2" fill="1" visible="no" active="no"/>
+<layer number="19" name="Unrouted" color="6" fill="1" visible="no" active="no"/>
+<layer number="20" name="Dimension" color="15" fill="1" visible="no" active="no"/>
+<layer number="21" name="tPlace" color="7" fill="1" visible="no" active="no"/>
+<layer number="22" name="bPlace" color="7" fill="1" visible="no" active="no"/>
+<layer number="23" name="tOrigins" color="15" fill="1" visible="no" active="no"/>
+<layer number="24" name="bOrigins" color="15" fill="1" visible="no" active="no"/>
+<layer number="25" name="tNames" color="7" fill="1" visible="no" active="no"/>
+<layer number="26" name="bNames" color="7" fill="1" visible="no" active="no"/>
+<layer number="27" name="tValues" color="7" fill="1" visible="no" active="no"/>
+<layer number="28" name="bValues" color="7" fill="1" visible="no" active="no"/>
 <layer number="29" name="tStop" color="7" fill="3" visible="no" active="no"/>
 <layer number="30" name="bStop" color="7" fill="6" visible="no" active="no"/>
@@
 <layer number="35" name="tGlue" color="7" fill="4" visible="no" active="no"/>
 <layer number="36" name="bGlue" color="7" fill="5" visible="no" active="no"/>
-<layer number="37" name="tTest" color="7" fill="1" visible="yes" active="no"/>
-<layer number="38" name="bTest" color="7" fill="1" visible="yes" active="no"/>
+<layer number="37" name="tTest" color="7" fill="1" visible="no" active="no"/>
+<layer number="38" name="bTest" color="7" fill="1" visible="no" active="no"/>
 <layer number="39" name="tKeepout" color="4" fill="11" visible="no" active="no"/>
 <layer number="40" name="bKeepout" color="1" fill="11" visible="no" active="no"/>
@@
 <layer number="44" name="Drills" color="7" fill="1" visible="no" active="no"/>
 <layer number="45" name="Holes" color="7" fill="1" visible="no" active="no"/>
-<layer number="46" name="Milling" color="3" fill="1" visible="yes" active="no"/>
-<layer number="47" name="Measures" color="7" fill="1" visible="yes" active="no"/>
-<layer number="48" name="Document" color="7" fill="1" visible="yes" active="no"/>
-<layer number="49" name="Reference" color="7" fill="1" visible="yes" active="no"/>
-<layer number="50" name="dxf" color="7" fill="1" visible="yes" active="no"/>
-<layer number="51" name="tDocu" color="7" fill="1" visible="yes" active="no"/>
-<layer number="52" name="bDocu" color="7" fill="1" visible="yes" active="no"/>
-<layer number="53" name="tGND_GNDA" color="7" fill="9" visible="yes" active="no"/>
-<layer number="54" name="bGND_GNDA" color="1" fill="9" visible="yes" active="no"/>
-<layer number="56" name="wert" color="7" fill="1" visible="yes" active="no"/>
+<layer number="46" name="Milling" color="3" fill="1" visible="no" active="no"/>
+<layer number="47" name="Measures" color="7" fill="1" visible="no" active="no"/>
+<layer number="48" name="Document" color="7" fill="1" visible="no" active="no"/>
+<layer number="49" name="Reference" color="7" fill="1" visible="no" active="no"/>
+<layer number="50" name="dxf" color="7" fill="1" visible="no" active="no"/>
+<layer number="51" name="tDocu" color="7" fill="1" visible="no" active="no"/>
+<layer number="52" name="bDocu" color="7" fill="1" visible="no" active="no"/>
+<layer number="53" name="tGND_GNDA" color="7" fill="9" visible="no" active="no"/>
+<layer number="54" name="bGND_GNDA" color="1" fill="9" visible="no" active="no"/>
+<layer number="56" name="wert" color="7" fill="1" visible="no" active="no"/>
 <layer number="91" name="Nets" color="2" fill="1" visible="yes" active="yes"/>
 <layer number="92" name="Busses" color="1" fill="1" visible="yes" active="yes"/>
@@
 <part name="C5" library="rcl" deviceset="C-EU" device="C0603K"/>
 <part name="J2" library="dp_devices" deviceset="CON_HEADER_1X04" device=""/>
+<part name="GND7" library="supply1" deviceset="GND" device=""/>
 </parts>
 <sheets>
@@
 <instance part="C5" gate="G$1" x="-38.1" y="63.5" rot="R270"/>
 <instance part="J2" gate="J" x="86.36" y="60.96"/>
+<instance part="GND7" gate="1" x="147.32" y="124.46"/>
 </instances>
 <busses>
@@
 <pinref part="GND6" gate="1" pin="GND"/>
 </segment>
+<segment>
+<pinref part="U$4" gate="G$1" pin="PIO5"/>
+<pinref part="GND7" gate="1" pin="GND"/>
+<wire x1="142.24" y1="132.08" x2="147.32" y2="132.08" width="0.1524" layer="91"/>
+<wire x1="147.32" y1="132.08" x2="147.32" y2="127" width="0.1524" layer="91"/>
+</segment>
 </net>

Commit message: routing done.Optimize before printing
Connections:
- net +3V3: now also IC2.VCC@2
- net GND: now also IC2.GND@2
Changed lines of the file:
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@@
 <?xml version="1.0" encoding="utf-8"?>
 <!DOCTYPE eagle SYSTEM "eagle.dtd">
-<eagle version="6.1">
+<eagle version="6.2">
 <drawing>
 <settings>
@@
 <wire x1="-43.18" y1="63.5" x2="-43.18" y2="45.72" width="0.1524" layer="91"/>
 <wire x1="-43.18" y1="45.72" x2="-30.48" y2="45.72" width="0.1524" layer="91"/>
+<pinref part="IC2" gate="G$1" pin="GND@2"/>
+<wire x1="-17.78" y1="48.26" x2="-22.86" y2="48.26" width="0.1524" layer="91"/>
+<wire x1="-22.86" y1="48.26" x2="-22.86" y2="50.8" width="0.1524" layer="91"/>
 </segment>
 <segment>
@@
 </segment>
 <segment>
-<wire x1="-20.32" y1="27.94" x2="-20.32" y2="45.72" width="0.1524" layer="91"/>
+<wire x1="-20.32" y1="27.94" x2="-20.32" y2="43.18" width="0.1524" layer="91"/>
+<wire x1="-20.32" y1="43.18" x2="-20.32" y2="45.72" width="0.1524" layer="91"/>
 <wire x1="-20.32" y1="45.72" x2="-17.78" y2="45.72" width="0.1524" layer="91"/>
 <wire x1="-22.86" y1="45.72" x2="-20.32" y2="45.72" width="0.1524" layer="91"/>
@@
 <pinref part="C1" gate="G$1" pin="2"/>
 <pinref part="IC2" gate="G$1" pin="VCC@1"/>
-</segment>
-<segment>
+<pinref part="IC2" gate="G$1" pin="VCC@2"/>
+<wire x1="-17.78" y1="43.18" x2="-20.32" y2="43.18" width="0.1524" layer="91"/>
+<junction x="-20.32" y="43.18"/>
+</segment>
+<segment>

Commit message: schematic inconsistency with board issue resolved
Parts:
- removed U1: (no value), microbuilder:LM1117SOT223-WAVE
- added IC1: (no value), SparkFun:V_REG_LM1117SOT223
- J1: value (none) -> POWER_JACKSLT; device con-jack:DCJ0303 -> SparkFun:POWER_JACKSLT
Connections:
- net +3V3: now also IC1.OUT, IC1.OUT@1; no longer IC2.VCC@2, U1.OUT
- net 12V: now also IC1.IN, J1.GND, J1.GNDBREAK; no longer J1.2, J1.3, U1.IN
- net GND: now also IC1.ADJ, J1.PWR; no longer J1.1, U1.ADJ
Changed lines of the file:
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@@
 <?xml version="1.0" encoding="utf-8"?>
 <!DOCTYPE eagle SYSTEM "eagle.dtd">
-<eagle version="6.2">
+<eagle version="6.1">
 <drawing>
 <settings>
@@
 </classes>
 <parts>
-<part name="U1" library="microbuilder" deviceset="LM1117" device="SOT223-WAVE"/>
 <part name="+3V1" library="supply1" deviceset="+3V3" device=""/>
 <part name="GND1" library="supply1" deviceset="GND" device=""/>
-<part name="J1" library="con-jack" deviceset="DCJ0303" device=""/>
 <part name="GND2" library="supply1" deviceset="GND" device=""/>
 <part name="GND3" library="supply1" deviceset="GND" device=""/>
-<part name="U$1" library="microbuilder" deviceset="12V" device=""/>
 <part name="U$2" library="microbuilder" deviceset="12V" device=""/>
 <part name="+3V2" library="supply1" deviceset="+3V3" device=""/>
@@
 <part name="IC2" library="atmel" deviceset="MEGA8" device="-AI"/>
 <part name="SW1" library="dp_devices" deviceset="SW_TACT_4P" device=""/>
-<part name="C2" library="dp_devices" deviceset="CAPACITOR_POL" device="-SMC_A" value="10uF"/>
 <part name="C3" library="dp_devices" deviceset="CAPACITOR_POL" device="-SMC_A" value="10uF"/>
 <part name="Y1" library="SparkFun" deviceset="CRYSTAL" device="SMD"/>
@@
 <part name="J2" library="dp_devices" deviceset="CON_HEADER_1X04" device=""/>
 <part name="GND7" library="supply1" deviceset="GND" device=""/>
+<part name="IC1" library="SparkFun" deviceset="V_REG_LM1117" device="SOT223"/>
+<part name="C2" library="dp_devices" deviceset="CAPACITOR_POL" device="-SMC_A" value="10uF"/>
+<part name="J1" library="SparkFun" deviceset="POWER_JACK" device="SLT"/>
+<part name="U$3" library="microbuilder" deviceset="12V" device=""/>
 </parts>
 <sheets>
@@
 </plain>
 <instances>
-<instance part="U1" gate="G$1" x="53.34" y="111.76"/>
 <instance part="+3V1" gate="G$1" x="63.5" y="121.92"/>
 <instance part="GND1" gate="1" x="53.34" y="81.28"/>
-<instance part="J1" gate="G$1" x="17.78" y="109.22"/>
 <instance part="GND2" gate="1" x="30.48" y="119.38" rot="R180"/>
 <instance part="GND3" gate="1" x="66.04" y="17.78"/>
-<instance part="U$1" gate="G$1" x="43.18" y="124.46"/>
 <instance part="U$2" gate="G$1" x="91.44" y="45.72"/>
 <instance part="+3V2" gate="G$1" x="-20.32" y="25.4" rot="R180"/>
@@
 <instance part="IC2" gate="G$1" x="5.08" y="55.88"/>
 <instance part="SW1" gate="G$1" x="15.24" y="88.9"/>
-<instance part="C2" gate="C" x="43.18" y="104.14"/>
 <instance part="C3" gate="C" x="63.5" y="104.14"/>
 <instance part="Y1" gate="G$1" x="-30.48" y="60.96" rot="R90"/>
@@
 <instance part="J2" gate="J" x="86.36" y="60.96"/>
 <instance part="GND7" gate="1" x="147.32" y="124.46"/>
+<instance part="IC1" gate="G$1" x="53.34" y="111.76"/>
+<instance part="C2" gate="C" x="43.18" y="104.14"/>
+<instance part="J1" gate="G$1" x="22.86" y="104.14"/>
+<instance part="U$3" gate="G$1" x="43.18" y="124.46"/>
 </instances>
 <busses>
@@
 <segment>
 <wire x1="53.34" y1="104.14" x2="53.34" y2="99.06" width="0.1524" layer="91"/>
-<pinref part="U1" gate="G$1" pin="ADJ"/>
 <pinref part="GND1" gate="1" pin="GND"/>
-<pinref part="C2" gate="C" pin="-"/>
 <wire x1="53.34" y1="99.06" x2="53.34" y2="83.82" width="0.1524" layer="91"/>
-<wire x1="43.18" y1="99.06" x2="53.34" y2="99.06" width="0.1524" layer="91"/>
 <pinref part="C3" gate="C" pin="-"/>
 <wire x1="53.34" y1="99.06" x2="63.5" y2="99.06" width="0.1524" layer="91"/>
 <junction x="53.34" y="99.06"/>
+<wire x1="43.18" y1="99.06" x2="53.34" y2="99.06" width="0.1524" layer="91"/>
+<pinref part="IC1" gate="G$1" pin="ADJ"/>
+<pinref part="C2" gate="C" pin="-"/>
 </segment>
 <segment>
 <wire x1="25.4" y1="111.76" x2="30.48" y2="111.76" width="0.1524" layer="91"/>
 <wire x1="30.48" y1="111.76" x2="30.48" y2="116.84" width="0.1524" layer="91"/>
-<pinref part="J1" gate="G$1" pin="1"/>
 <pinref part="GND2" gate="1" pin="GND"/>
+<pinref part="J1" gate="G$1" pin="PWR"/>
 </segment>
 <segment>
@@
 <wire x1="60.96" y1="111.76" x2="63.5" y2="111.76" width="0.1524" layer="91"/>
 <wire x1="63.5" y1="111.76" x2="63.5" y2="119.38" width="0.1524" layer="91"/>
-<pinref part="U1" gate="G$1" pin="OUT"/>
 <pinref part="+3V1" gate="G$1" pin="+3V3"/>
 <pinref part="C3" gate="C" pin="+"/>
 <wire x1="63.5" y1="111.76" x2="63.5" y2="106.68" width="0.1524" layer="91"/>
 <junction x="63.5" y="111.76"/>
-</segment>
-<segment>
-<wire x1="-20.32" y1="27.94" x2="-20.32" y2="43.18" width="0.1524" layer="91"/>
-<wire x1="-20.32" y1="43.18" x2="-20.32" y2="45.72" width="0.1524" layer="91"/>
+<pinref part="IC1" gate="G$1" pin="OUT"/>
+<pinref part="IC1" gate="G$1" pin="OUT@1"/>
+<wire x1="60.96" y1="109.22" x2="60.96" y2="111.76" width="0.1524" layer="91"/>
+</segment>
+<segment>
+<wire x1="-20.32" y1="27.94" x2="-20.32" y2="45.72" width="0.1524" layer="91"/>
 <wire x1="-20.32" y1="45.72" x2="-17.78" y2="45.72" width="0.1524" layer="91"/>
 <wire x1="-22.86" y1="45.72" x2="-20.32" y2="45.72" width="0.1524" layer="91"/>
@@
 <pinref part="C1" gate="G$1" pin="2"/>
 <pinref part="IC2" gate="G$1" pin="VCC@1"/>
-<pinref part="IC2" gate="G$1" pin="VCC@2"/>
-<wire x1="-17.78" y1="43.18" x2="-20.32" y2="43.18" width="0.1524" layer="91"/>
-<junction x="-20.32" y="43.18"/>
 </segment>
 <segment>
@@
 <net name="12V" class="0">
 <segment>
+<wire x1="86.36" y1="55.88" x2="81.28" y2="55.88" width="0.1524" layer="91"/>
+<wire x1="81.28" y1="55.88" x2="81.28" y2="45.72" width="0.1524" layer="91"/>
+<wire x1="81.28" y1="45.72" x2="91.44" y2="45.72" width="0.1524" layer="91"/>
+<pinref part="U$2" gate="G$1" pin="12V"/>
+<pinref part="J2" gate="J" pin="4"/>
+</segment>
+<segment>
 <wire x1="25.4" y1="109.22" x2="25.4" y2="106.68" width="0.1524" layer="91"/>
 <wire x1="25.4" y1="106.68" x2="38.1" y2="106.68" width="0.1524" layer="91"/>
@@
 <wire x1="43.18" y1="111.76" x2="43.18" y2="124.46" width="0.1524" layer="91"/>
 <junction x="43.18" y="111.76"/>
-<pinref part="J1" gate="G$1" pin="2"/>
-<pinref part="J1" gate="G$1" pin="3"/>
-<pinref part="U1" gate="G$1" pin="IN"/>
-<pinref part="U$1" gate="G$1" pin="12V"/>
+<wire x1="43.18" y1="111.76" x2="43.18" y2="106.68" width="0.1524" layer="91"/>
+<pinref part="IC1" gate="G$1" pin="IN"/>
 <pinref part="C2" gate="C" pin="+"/>
-<wire x1="43.18" y1="111.76" x2="43.18" y2="106.68" width="0.1524" layer="91"/>
-</segment>
-<segment>
-<wire x1="86.36" y1="55.88" x2="81.28" y2="55.88" width="0.1524" layer="91"/>
-<wire x1="81.28" y1="55.88" x2="81.28" y2="45.72" width="0.1524" layer="91"/>
-<wire x1="81.28" y1="45.72" x2="91.44" y2="45.72" width="0.1524" layer="91"/>
-<pinref part="U$2" gate="G$1" pin="12V"/>
-<pinref part="J2" gate="J" pin="4"/>
-</segment>
-</net>
+<pinref part="J1" gate="G$1" pin="GNDBREAK"/>
+<pinref part="J1" gate="G$1" pin="GND"/>
+<junction x="25.4" y="106.68"/>
+<pinref part="U$3" gate="G$1" pin="12V"/>
+</segment>
+</net>

Commit message: barrel jack was connected in reverse. corrected now.
Connections:
- net 12V: now also J1.PWR; no longer J1.GND, J1.GNDBREAK
- net GND: now also J1.GND, J1.GNDBREAK; no longer J1.PWR
Changed lines of the file:
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@@
 <instance part="+3V1" gate="G$1" x="63.5" y="121.92"/>
 <instance part="GND1" gate="1" x="53.34" y="81.28"/>
-<instance part="GND2" gate="1" x="30.48" y="119.38" rot="R180"/>
+<instance part="GND2" gate="1" x="30.48" y="101.6"/>
 <instance part="GND3" gate="1" x="66.04" y="17.78"/>
 <instance part="U$2" gate="G$1" x="91.44" y="45.72"/>
@@
 </segment>
 <segment>
-<wire x1="25.4" y1="111.76" x2="30.48" y2="111.76" width="0.1524" layer="91"/>
-<wire x1="30.48" y1="111.76" x2="30.48" y2="116.84" width="0.1524" layer="91"/>
-<pinref part="GND2" gate="1" pin="GND"/>
-<pinref part="J1" gate="G$1" pin="PWR"/>
-</segment>
-<segment>
 <wire x1="63.5" y1="22.86" x2="66.04" y2="22.86" width="0.1524" layer="91"/>
 <wire x1="66.04" y1="22.86" x2="66.04" y2="20.32" width="0.1524" layer="91"/>
@@
 <wire x1="147.32" y1="132.08" x2="147.32" y2="127" width="0.1524" layer="91"/>
 </segment>
+<segment>
+<pinref part="J1" gate="G$1" pin="GNDBREAK"/>
+<pinref part="J1" gate="G$1" pin="GND"/>
+<wire x1="25.4" y1="109.22" x2="25.4" y2="106.68" width="0.1524" layer="91"/>
+<pinref part="GND2" gate="1" pin="GND"/>
+<wire x1="25.4" y1="106.68" x2="30.48" y2="106.68" width="0.1524" layer="91"/>
+<wire x1="30.48" y1="106.68" x2="30.48" y2="104.14" width="0.1524" layer="91"/>
+</segment>
 </net>
 <net name="+3V3" class="0">
@@
 </segment>
 <segment>
-<wire x1="25.4" y1="109.22" x2="25.4" y2="106.68" width="0.1524" layer="91"/>
-<wire x1="25.4" y1="106.68" x2="38.1" y2="106.68" width="0.1524" layer="91"/>
-<wire x1="38.1" y1="106.68" x2="38.1" y2="111.76" width="0.1524" layer="91"/>
-<wire x1="38.1" y1="111.76" x2="43.18" y2="111.76" width="0.1524" layer="91"/>
 <wire x1="43.18" y1="111.76" x2="45.72" y2="111.76" width="0.1524" layer="91"/>
 <wire x1="43.18" y1="111.76" x2="43.18" y2="124.46" width="0.1524" layer="91"/>
@@
 <pinref part="IC1" gate="G$1" pin="IN"/>
 <pinref part="C2" gate="C" pin="+"/>
-<pinref part="J1" gate="G$1" pin="GNDBREAK"/>
-<pinref part="J1" gate="G$1" pin="GND"/>
-<junction x="25.4" y="106.68"/>
 <pinref part="U$3" gate="G$1" pin="12V"/>
-</segment>
-</net>
+<pinref part="J1" gate="G$1" pin="PWR"/>
+<wire x1="25.4" y1="111.76" x2="43.18" y2="111.76" width="0.1524" layer="91"/>
+</segment>
+</net>
